File: sense_pcb/_saved_sense_pcb.sch (KiCad schematic (older format))
At the start: 31 parts, among them J1 Conn_02x06_Odd_Even, U1 DRV5053VAQDBZR, U10 DRV5053VAQDBZR, U11 DRV5053VAQDBZR, U12 DRV5053VAQDBZR, U13 DRV5053VAQDBZR, U14 4051, U15 DRV5053VAQDBZR, U16 DRV5053VAQDBZR, U17 DRV5053VAQDBZR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

Commit message: adds netlist and pcb
Parts:
- C1, C2, C3: footprint (none) -> Capacitors_SMD:C_1206_HandSoldering
- J1: footprint (none) -> Pin_Headers:Pin_Header_Straight_2x06_Pitch2.54mm
- U14, U23, U5: footprint (none) -> SMD_Packages:SO-16-N
Changed lines of the file:
@@
 F 0 "U5" H 1775 2900 50  0000 C CNN
 F 1 "4051" H 1775 2700 50  0000 C CNN
-F 2 "" H 1675 2900 60  0001 C CNN
+F 2 "SMD_Packages:SO-16-N" H 1675 2900 60  0001 C CNN
 F 3 "" H 1675 2900 60  0001 C CNN
 	1    1675 2900
@@
 F 0 "C1" H 2600 2725 50  0000 L CNN
 F 1 "C" H 2600 2525 50  0000 L CNN
-F 2 "" H 2613 2475 50  0001 C CNN
+F 2 "Capacitors_SMD:C_1206_HandSoldering" H 2613 2475 50  0001 C CNN
 F 3 "" H 2575 2625 50  0001 C CNN
 	1    2575 2625
@@
 F 0 "U14" H 3750 2900 50  0000 C CNN
 F 1 "4051" H 3750 2700 50  0000 C CNN
-F 2 "" H 3650 2900 60  0001 C CNN
+F 2 "SMD_Packages:SO-16-N" H 3650 2900 60  0001 C CNN
 F 3 "" H 3650 2900 60  0001 C CNN
 	1    3650 2900
@@
 F 0 "C2" H 4575 2725 50  0000 L CNN
 F 1 "C" H 4575 2525 50  0000 L CNN
-F 2 "" H 4588 2475 50  0001 C CNN
+F 2 "Capacitors_SMD:C_1206_HandSoldering" H 4588 2475 50  0001 C CNN
 F 3 "" H 4550 2625 50  0001 C CNN
 	1    4550 2625
@@
 F 0 "U23" H 5600 2900 50  0000 C CNN
 F 1 "4051" H 5600 2700 50  0000 C CNN
-F 2 "" H 5500 2900 60  0001 C CNN
+F 2 "SMD_Packages:SO-16-N" H 5500 2900 60  0001 C CNN
 F 3 "" H 5500 2900 60  0001 C CNN
 	1    5500 2900
@@
 F 0 "C3" H 6425 2725 50  0000 L CNN
 F 1 "C" H 6425 2525 50  0000 L CNN
-F 2 "" H 6438 2475 50  0001 C CNN
+F 2 "Capacitors_SMD:C_1206_HandSoldering" H 6438 2475 50  0001 C CNN
 F 3 "" H 6400 2625 50  0001 C CNN
 	1    6400 2625
@@
 F 0 "J1" H 3425 1250 50  0000 C CNN
 F 1 "Conn_02x06_Odd_Even" H 3425 550 50  0000 C CNN
-F 2 "" H 3375 950 50  0001 C CNN
+F 2 "Pin_Headers:Pin_Header_Straight_2x06_Pitch2.54mm" H 3375 950 50  0001 C CNN
 F 3 "" H 3375 950 50  0001 C CNN
 	1    3375 950

Commit message: adds measurements
Connections:
- net VDD is gone; now on net VCC: U14.16 (VDD), U23.16 (VDD), U5.16 (VDD)
- net VSS is gone; now on net GND: U14.8 (VSS), U23.8 (VSS), U5.8 (VSS)
Changed lines of the file:
@@
 Connection ~ 6275 2200
 Connection ~ 5850 4375
+$Comp
+L VCC #PWR09
+U 1 1 5C7A43BC
+P 975 825
+F 0 "#PWR09" H 975 675 50  0001 C CNN
+F 1 "VCC" H 975 975 50  0000 C CNN
+F 2 "" H 975 825 50  0001 C CNN
+F 3 "" H 975 825 50  0001 C CNN
+	1    975  825
+	1    0    0    -1
+$EndComp
+$Comp
+L GND #PWR010
+U 1 1 5C7A440E
+P 975 1250
+F 0 "#PWR010" H 975 1000 50  0001 C CNN
+F 1 "GND" H 975 1100 50  0000 C CNN
+F 2 "" H 975 1250 50  0001 C CNN
+F 3 "" H 975 1250 50  0001 C CNN
+	1    975  1250
+	1    0    0    -1
+$EndComp
+$Comp
+L VDD #PWR011
+U 1 1 5C7A4460
+P 1150 825
+F 0 "#PWR011" H 1150 675 50  0001 C CNN
+F 1 "VDD" H 1150 975 50  0000 C CNN
+F 2 "" H 1150 825 50  0001 C CNN
+F 3 "" H 1150 825 50  0001 C CNN
+	1    1150 825
+	1    0    0    -1
+$EndComp
+$Comp
+L VSS #PWR012
+U 1 1 5C7A44B2
+P 1150 1250
+F 0 "#PWR012" H 1150 1100 50  0001 C CNN
+F 1 "VSS" H 1150 1400 50  0000 C CNN
+F 2 "" H 1150 1250 50  0001 C CNN
+F 3 "" H 1150 1250 50  0001 C CNN
+	1    1150 1250
+	1    0    0    -1
+$EndComp
+Wire Wire Line
+	975  1250 1150 1250
+Wire Wire Line
+	1150 825  975  825
 $EndSCHEMATC
